Commit message: Add package name parameter and split xarm7 XML

File: src/xarm7_sim_config/description/mujoco.ros2_control.xacro (robot description, xacro)
@@ -1,5 +1,5 @@
 <?xml version="1.0" encoding="utf-8"?>
 <robot xmlns:xacro="http://ros.org/wiki/xacro">
-  <xacro:macro name="xarm7_mujoco_ros2_control" params="prefix:='' mujoco_model mujoco_viewer:=false
+  <xacro:macro name="xarm7_mujoco_ros2_control" params="prefix:='' mujoco_model mujoco_model_package mujoco_viewer:=false
     joint1_lower_limit:=${-2.0*pi}  joint1_upper_limit:=${2.0*pi}
     joint2_lower_limit:=${-2.059}  joint2_upper_limit:=${2.0944}
@@ -13,5 +13,5 @@
           <plugin>picknik_mujoco_ros/MujocoSystem</plugin>
           <param name="mujoco_model">${mujoco_model}</param>
-          <param name="mujoco_model_package">xarm7_sim_config</param>
+          <param name="mujoco_model_package">${mujoco_model_package}</param>
           <param name="render_publish_rate">20</param>
           <param name="tf_publish_rate">60</param>

File: src/xarm7_sim_config/description/picknik_xarm.xacro (robot description, xacro)
@@ -39,5 +39,5 @@
     <xacro:include filename="$(find xarm7_sim_config)/description/mujoco.ros2_control.xacro" />
     <xacro:xarm7_mujoco_ros2_control
-      mujoco_model="description/mujoco/scene.xml" mujoco_viewer="false"
+      mujoco_model="description/mujoco/scene.xml" mujoco_viewer="false" mujoco_model_package="xarm7_sim_config"
     />
   </xacro:if>
