Commit message: Add pose jog frame and cleanup configs

File: src/xarm7_sim_config/description/picknik_xarm.xacro (robot description, xacro)
@@ -36,4 +36,10 @@
   >
   </xacro:picknik_xarm>
+  <link name="link_pose_jog"/>
+  <joint name="joint_pose_jog" type="fixed">
+    <origin xyz="0 0 0" rpy="0 0 -1.57079632679" />
+    <parent link="link_eef" />
+    <child link="link_pose_jog" />
+  </joint>
   <xacro:if value="$(arg launch_mujoco)">
     <xacro:include filename="$(find xarm7_sim_config)/description/mujoco.ros2_control.xacro" />

File: src/xarm7_sim_config/description/picknik_xarm_macro.xacro (robot description, xacro)
@@ -3,5 +3,5 @@
   <xacro:macro
     name="picknik_xarm"
-    params="attach_to launch_ros2_control"
+    params="attach_to attach_xyz:='0 0 0' attach_rpy:='0 0 0' launch_ros2_control"
   >
     <!-- parameters -->

File: src/xarm_base_config/description/picknik_xarm.xacro (robot description, xacro)
@@ -33,3 +33,9 @@
   >
   </xacro:picknik_xarm>
+  <link name="link_pose_jog"/>
+  <joint name="joint_pose_jog" type="fixed">
+    <origin xyz="0 0 0" rpy="0 0 -1.57079632679" />
+    <parent link="link_eef" />
+    <child link="link_pose_jog" />
+  </joint>
 </robot>

File: src/xarm_base_config/description/picknik_xarm_macro.xacro (robot description, xacro)
@@ -3,5 +3,5 @@
   <xacro:macro
     name="picknik_xarm"
-    params="attach_to"
+    params="attach_to attach_xyz:='0 0 0' attach_rpy:='0 0 0'"
   >
     <!-- parameters -->

Commit message: Update xacro passthrough

File: src/xarm7_sim_config/description/picknik_xarm.xacro (robot description, xacro)
@@ -32,14 +32,10 @@
   <!-- Robot: contains robot description from the world frame to the tool frame -->
   <xacro:picknik_xarm
-    attach_to="world"
+    attach_to="$(arg attach_to)"
     launch_ros2_control= "$(arg launch_ros2_control)"
+    attach_xyz="$(arg attach_xyz)"
+    attach_rpy="$(arg attach_rpy)"
   >
   </xacro:picknik_xarm>
-  <link name="link_pose_jog"/>
-  <joint name="joint_pose_jog" type="fixed">
-    <origin xyz="0 0 0" rpy="0 0 -1.57079632679" />
-    <parent link="link_eef" />
-    <child link="link_pose_jog" />
-  </joint>
   <xacro:if value="$(arg launch_mujoco)">
     <xacro:include filename="$(find xarm7_sim_config)/description/mujoco.ros2_control.xacro" />

File: src/xarm7_sim_config/description/picknik_xarm_macro.xacro (robot description, xacro)
@@ -3,67 +3,75 @@
   <xacro:macro
     name="picknik_xarm"
-    params="attach_to attach_xyz:='0 0 0' attach_rpy:='0 0 0' launch_ros2_control"
+    params="
+    prefix:=''
+    hw_ns:='xarm'
+    limited:=false
+    effort_control:=false
+    velocity_control:=false
+    add_gripper:=false
+    add_vacuum_gripper:=false
+    add_bio_gripper:=false
+    model1300:=false
+    dof:=7
+    robot_ip:=''
+    robot_type:='xarm'
+    robot_sn:=''
+    report_type:='normal'
+    launch_ros2_control:='true'
+    ros2_control_plugin:='uf_robot_hardware/UFRobotSystemHardware'
+    ros2_control_params:=''
+    add_realsense_d435i:=false
+    add_d435i_links:=true
+    use_gazebo_camera:=false
+    add_other_geometry:=false
+    geometry_type:='box'
+    geometry_mass:='0.1'
+    geometry_radius:='0.1'
+    geometry_height:='0.1'
+    geometry_length:='0.1'
+    geometry_width:='0.1'
+    geometry_mesh_filename:=''
+    geometry_mesh_origin_xyz:='0 0 0'
+    geometry_mesh_origin_rpy:='0 0 0'
+    geometry_mesh_tcp_xyz:='0 0 0'
+    geometry_mesh_tcp_rpy:='0 0 0'
+    baud_checkset:=true
+    default_gripper_baud:=2000000
+    attach_to:='world'
+    attach_xyz:='0 0 0'
+    attach_rpy:='0 0 0'
+    mesh_suffix:='stl'
+    kinematics_suffix:=''
+    "
   >
-    <!-- parameters -->
-    <xacro:arg name="prefix" default=""/>
-    <xacro:arg name="hw_ns" default="xarm"/>
-    <xacro:arg name="limited" default="false"/>
-    <xacro:arg name="effort_control" default="false"/>
-    <xacro:arg name="velocity_control" default="false"/>
-    <xacro:arg name="add_gripper" default="false"/>
-    <xacro:arg name="add_vacuum_gripper" default="false"/>
-    <xacro:arg name="add_bio_gripper" default="false"/>
-    <xacro:arg name="model1300" default="false"/>
-    <xacro:arg name="dof" default="7"/>
-    <xacro:arg name="robot_ip" default=""/>
-    <xacro:arg name="robot_type" default="xarm"/>
-    <xacro:arg name="robot_sn" default=""/>
-    <xacro:arg name="report_type" default="normal"/>
-    <xacro:arg name="launch_ros2_control" default="true"/>
-    <xacro:arg name="ros2_control_plugin" default="uf_robot_hardware/UFRobotSystemHardware"/>
-    <xacro:arg name="ros2_control_params" default=""/>
-    <xacro:arg name="add_realsense_d435i" default="false"/>
-    <xacro:arg name="add_d435i_links" default="true"/>
-    <xacro:arg name="use_gazebo_camera" default="false"/>
-    <xacro:arg name="add_other_geometry" default="false"/>
-    <xacro:arg name="geometry_type" default="box"/>
-    <xacro:arg name="geometry_mass" default="0.1"/>
-    <xacro:arg name="geometry_height" default="0.1"/>
-    <xacro:arg name="geometry_radius" default="0.1"/>
-    <xacro:arg name="geometry_length" default="0.1"/>
-    <xacro:arg name="geometry_width" default="0.1"/>
-    <xacro:arg name="geometry_mesh_filename" default=""/>
-    <xacro:arg name="geometry_mesh_origin_xyz" default="0 0 0"/>
-    <xacro:arg name="geometry_mesh_origin_rpy" default="0 0 0"/>
-    <xacro:arg name="geometry_mesh_tcp_xyz" default="0 0 0"/>
-    <xacro:arg name="geometry_mesh_tcp_rpy" default="0 0 0"/>
-    <xacro:arg name="baud_checkset" default="true"/>
-    <xacro:arg name="default_gripper_baud" default="2000000"/>
-    <xacro:arg name="attach_to" default="world"/>
-    <xacro:arg name="attach_xyz" default="0 0 0"/>
-    <xacro:arg name="attach_rpy" default="0 0 0"/>
     <xacro:arg name="mesh_suffix" default="stl"/>
     <xacro:arg name="kinematics_suffix" default=""/>
     <!-- load xarm device -->
     <xacro:include filename="$(find xarm7_sim_config)/description/xarm_device_macro.xacro" />
-    <xacro:xarm_device prefix="$(arg prefix)" hw_ns="$(arg hw_ns)" limited="$(arg limited)"
-      effort_control="$(arg effort_control)" velocity_control="$(arg velocity_control)"
-      add_gripper="$(arg add_gripper)" add_vacuum_gripper="$(arg add_vacuum_gripper)"
-      add_bio_gripper="$(arg add_bio_gripper)" dof="$(arg dof)" launch_ros2_control= "$(arg launch_ros2_control)"
-      ros2_control_plugin="$(arg ros2_control_plugin)" robot_type="$(arg robot_type)"
-      load_gazebo_plugin="true" ros2_control_params="$(arg ros2_control_params)"
-      add_realsense_d435i="$(arg add_realsense_d435i)"
-      add_d435i_links="$(arg add_d435i_links)"
-      add_other_geometry="$(arg add_other_geometry)"
-      geometry_type="$(arg geometry_type)" geometry_mass="$(arg geometry_mass)"
-      geometry_height="$(arg geometry_height)" geometry_radius="$(arg geometry_radius)"
-      geometry_length="$(arg geometry_length)" geometry_width="$(arg geometry_width)"
-      geometry_mesh_filename="$(arg geometry_mesh_filename)"
-      geometry_mesh_origin_xyz="$(arg geometry_mesh_origin_xyz)" geometry_mesh_origin_rpy="$(arg geometry_mesh_origin_rpy)"
-      geometry_mesh_tcp_xyz="$(arg geometry_mesh_tcp_xyz)" geometry_mesh_tcp_rpy="$(arg geometry_mesh_tcp_rpy)"
-      robot_ip="$(arg robot_ip)" report_type="$(arg report_type)"
-      baud_checkset="$(arg baud_checkset)" default_gripper_baud="$(arg default_gripper_baud)"
-      model1300="$(arg model1300)" attach_to="$(arg attach_to)" attach_xyz="$(arg attach_xyz)" attach_rpy="$(arg attach_rpy)"
-      robot_sn="$(arg robot_sn)" use_gazebo_camera="$(arg use_gazebo_camera)" mesh_suffix="$(arg mesh_suffix)" kinematics_suffix="$(arg kinematics_suffix)" />
+    <xacro:xarm_device prefix="${prefix}" hw_ns="${hw_ns}" limited="${limited}"
+      effort_control="${effort_control}" velocity_control="${velocity_control}"
+      add_gripper="${add_gripper}" add_vacuum_gripper="${add_vacuum_gripper}"
+      add_bio_gripper="${add_bio_gripper}" dof="${dof}" launch_ros2_control= "${launch_ros2_control}"
+      ros2_control_plugin="${ros2_control_plugin}" robot_type="${robot_type}"
+      load_gazebo_plugin="true" ros2_control_params="${ros2_control_params}"
+      add_realsense_d435i="${add_realsense_d435i}"
+      add_d435i_links="${add_d435i_links}"
+      add_other_geometry="${add_other_geometry}"
+      geometry_type="${geometry_type}" geometry_mass="${geometry_mass}"
+      geometry_height="${geometry_height}" geometry_radius="${geometry_radius}"
+      geometry_length="${geometry_length}" geometry_width="${geometry_width}"
+      geometry_mesh_filename="${geometry_mesh_filename}"
+      geometry_mesh_origin_xyz="${geometry_mesh_origin_xyz}" geometry_mesh_origin_rpy="${geometry_mesh_origin_rpy}"
+      geometry_mesh_tcp_xyz="${geometry_mesh_tcp_xyz}" geometry_mesh_tcp_rpy="${geometry_mesh_tcp_rpy}"
+      robot_ip="${robot_ip}" report_type="${report_type}"
+      baud_checkset="${baud_checkset}" default_gripper_baud="${default_gripper_baud}"
+      model1300="${model1300}" attach_to="${attach_to}" attach_xyz="${attach_xyz}" attach_rpy="${attach_rpy}"
+      robot_sn="${robot_sn}" use_gazebo_camera="${use_gazebo_camera}" mesh_suffix="${mesh_suffix}" kinematics_suffix="${kinematics_suffix}" />
+    <link name="${prefix}link_pose_jog"/>
+    <joint name="${prefix}joint_pose_jog" type="fixed">
+      <origin xyz="0 0 0" rpy="0 0 -1.57079632679" />
+      <parent link="${prefix}link_eef" />
+      <child link="${prefix}link_pose_jog" />
+    </joint>
   </xacro:macro>
 </robot>
