Commit message: Add end_effector tag if there is no gripper (for iMarker teleop)

File: src/xarm_base_config/config/moveit/xarm.srdf.xacro (robot description, xacro)
@@ -16,3 +16,10 @@
       <joint name="joint_pose_jog" />
   </group>
+  <group name="gripper">
+      <link name="link_eef" />
+  </group>
+  <xacro:unless value="$(arg add_gripper)">
+    <!-- Add an end-effector tag for iMarker Teleoperation -->
+    <end_effector name="xarm_gripper" parent_link="link_eef" group="gripper" />
+  </xacro:unless>
 </robot>
